File: KicadFPGA.kicad_pcb (KiCad board)
At the start: 4 copper layers, 88.9 x 63.5 mm, 167 parts, among them J1 USB_B_Micro, J2 Conn_01x06_Male, J3 Conn_ARM_JTAG_SWD_10, J4 Conn_01x03_Male, J5 Conn_01x16_Male, Q1 FDV301N, Q2 FDV301N, Q3 FDV301N, Q4 FDV301N, Q5 FDV301N, U1 XC7A35T-FTG256, U2 Xilinx_FPGA_JTAG_Conn_2x7, U3 STM32F411CEUx, U4 MT25QU128, U5 TPS62142, U6 FT232RL, U7 TLV62084ADSGx, U8 TLV62084ADSGx, U9 SiT8008B, Y1 25MHz

Commit message: finished routing the thing
Parts:
- removed RX: LED_RX, digikey-footprints:0603
- removed TX: LED_TX, digikey-footprints:0603
- added D5: LED_RX, digikey-footprints:0603, F.Cu at (79.2, 120.8)
- added D6: LED_TX, digikey-footprints:0603, F.Cu at (79.2, 122.4)
- added G***: DaisyLogo3, KicadFPGA:DaisyLogo3, F.Cu at (134.8, 114.5)
- C63: value C -> 22uF
- TP1: value TestPoint -> tGND; footprint TestPoint:TestPoint_Pad_2.0x2.0mm -> TestPoint:TestPoint_Pad_1.0x1.0mm
- TP10: value TestPoint -> tFPGA_M1; footprint TestPoint:TestPoint_Pad_2.0x2.0mm -> TestPoint:TestPoint_Pad_1.0x1.0mm
- TP11: value TestPoint -> tFPGA_M2; footprint TestPoint:TestPoint_Pad_2.0x2.0mm -> TestPoint:TestPoint_Pad_1.0x1.0mm
- TP12: value TestPoint -> t5V; footprint TestPoint:TestPoint_Pad_2.0x2.0mm -> TestPoint:TestPoint_Pad_1.0x1.0mm
- TP13: value TestPoint -> tSPI_CS; footprint TestPoint:TestPoint_Pad_2.0x2.0mm -> TestPoint:TestPoint_Pad_1.0x1.0mm
- TP14: value TestPoint -> tSPI_SCK; footprint TestPoint:TestPoint_Pad_2.0x2.0mm -> TestPoint:TestPoint_Pad_1.0x1.0mm
- TP15: value TestPoint -> tSPI_MISO; footprint TestPoint:TestPoint_Pad_2.0x2.0mm -> TestPoint:TestPoint_Pad_1.0x1.0mm
- TP16: value TestPoint -> tSPI_MOSI; footprint TestPoint:TestPoint_Pad_2.0x2.0mm -> TestPoint:TestPoint_Pad_1.0x1.0mm
- TP17: value TestPoint -> tRXI; footprint TestPoint:TestPoint_Pad_2.0x2.0mm -> TestPoint:TestPoint_Pad_1.0x1.0mm
- TP18: value TestPoint -> tTXO; footprint TestPoint:TestPoint_Pad_2.0x2.0mm -> TestPoint:TestPoint_Pad_1.0x1.0mm
- TP19: value TestPoint -> tJTAG_RST; footprint TestPoint:TestPoint_Pad_2.0x2.0mm -> TestPoint:TestPoint_Pad_1.0x1.0mm
- TP2: value TestPoint -> t3V3; footprint TestPoint:TestPoint_Pad_2.0x2.0mm -> TestPoint:TestPoint_Pad_1.0x1.0mm
- TP20: value TestPoint -> tJTAG_TCK; footprint TestPoint:TestPoint_Pad_2.0x2.0mm -> TestPoint:TestPoint_Pad_1.0x1.0mm
- TP21: value TestPoint -> tJTAG_TMS; footprint TestPoint:TestPoint_Pad_2.0x2.0mm -> TestPoint:TestPoint_Pad_1.0x1.0mm
- TP22: value TestPoint -> tJTAG_TDO; footprint TestPoint:TestPoint_Pad_2.0x2.0mm -> TestPoint:TestPoint_Pad_1.0x1.0mm
- TP23: value TestPoint -> tJTAG_TDI; footprint TestPoint:TestPoint_Pad_2.0x2.0mm -> TestPoint:TestPoint_Pad_1.0x1.0mm
- TP24: value TestPoint -> tBUS0; footprint TestPoint:TestPoint_Pad_2.0x2.0mm -> TestPoint:TestPoint_Pad_1.0x1.0mm
- TP25: value TestPoint -> tBUS1; footprint TestPoint:TestPoint_Pad_2.0x2.0mm -> TestPoint:TestPoint_Pad_1.0x1.0mm
- TP26: value TestPoint -> tBUS2; footprint TestPoint:TestPoint_Pad_2.0x2.0mm -> TestPoint:TestPoint_Pad_1.0x1.0mm
- TP27: value TestPoint -> tBUS3; footprint TestPoint:TestPoint_Pad_2.0x2.0mm -> TestPoint:TestPoint_Pad_1.0x1.0mm
- TP28: value TestPoint -> tBUS4; footprint TestPoint:TestPoint_Pad_2.0x2.0mm -> TestPoint:TestPoint_Pad_1.0x1.0mm
- TP29: value TestPoint -> tBUS5; footprint TestPoint:TestPoint_Pad_2.0x2.0mm -> TestPoint:TestPoint_Pad_1.0x1.0mm
- TP3: value TestPoint -> t1V8; footprint TestPoint:TestPoint_Pad_2.0x2.0mm -> TestPoint:TestPoint_Pad_1.0x1.0mm
- TP30: value TestPoint -> tBUS6; footprint TestPoint:TestPoint_Pad_2.0x2.0mm -> TestPoint:TestPoint_Pad_1.0x1.0mm
- TP31: value TestPoint -> tBUS7; footprint TestPoint:TestPoint_Pad_2.0x2.0mm -> TestPoint:TestPoint_Pad_1.0x1.0mm
- TP4: value TestPoint -> t1V0; footprint TestPoint:TestPoint_Pad_2.0x2.0mm -> TestPoint:TestPoint_Pad_1.0x1.0mm
- TP5: value TestPoint -> tFPGA_DONE; footprint TestPoint:TestPoint_Pad_2.0x2.0mm -> TestPoint:TestPoint_Pad_1.0x1.0mm
- TP6: value TestPoint -> tFPGA_INIT; footprint TestPoint:TestPoint_Pad_2.0x2.0mm -> TestPoint:TestPoint_Pad_1.0x1.0mm
- TP7: value TestPoint -> tFPGA_PROGRAM; footprint TestPoint:TestPoint_Pad_2.0x2.0mm -> TestPoint:TestPoint_Pad_1.0x1.0mm
- TP8: value TestPoint -> tFPGA_CCLK; footprint TestPoint:TestPoint_Pad_2.0x2.0mm -> TestPoint:TestPoint_Pad_1.0x1.0mm
- TP9: value TestPoint -> tFPGA_M0; footprint TestPoint:TestPoint_Pad_2.0x2.0mm -> TestPoint:TestPoint_Pad_1.0x1.0mm
- moved TP3 79.4 mm to (101.7, 119.1)
- moved TP12 71.3 mm to (95.9, 114.1)
- moved TP4 69.4 mm to (133.9, 128.8)
- moved TP2 65.6 mm to (93.9, 90.6)
- moved TP11 64.6 mm to (162.4, 127.0)
- moved TP16 63.3 mm to (150.2, 130.3)
- moved TP14 61.6 mm to (153.1, 122.5)
- moved TP5 59.9 mm to (123.9, 107.8)
- moved TP10 59.4 mm to (162.3, 119.3)
- moved TP15 58.7 mm to (145.4, 122.5)
- moved TP31 53.4 mm to (132.8, 118.0)
- moved TP30 53.1 mm to (130.9, 118.0)
- moved TP17 50.7 mm to (135.9, 111.5)
- moved TP29 49.5 mm to (127.5, 115.3)
- moved TP18 49.2 mm to (137.3, 114.9)
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Connections:
- U5 pad 15: +3V3 -> GND
- U5 pad 16: +3V3 -> GND
- U5 pad 17: +3V3 -> GND
- U5 pad 6: +3V3 -> GND
Routing:
- net +3V3: track 0.00 -> 450.4 mm, vias 0 -> 37
- net GND: track 0.00 -> 293.0 mm, vias 0 -> 50
- net +1V0: track 2.22 -> 121.8 mm, vias 0 -> 13
- net FPGA_BUTTON_1: track 0.00 -> 94.5 mm, vias 0 -> 2
- net FPGA_PROGRAM_B: track 0.00 -> 89.7 mm, vias 0 -> 4
- net FPGA_BUTTON_2: track 0.00 -> 86.0 mm, vias 0 -> 6
- net FT232_RXI: track 0.00 -> 84.0 mm, vias 0 -> 2
- net FT232_TXO: track 0.00 -> 83.8 mm, vias 0 -> 2
- net +1V8: track 0.00 -> 79.7 mm, vias 0 -> 6
- net +5V: track 34.9 -> 107.3 mm, vias 0 -> 1
- net M0_0: track 0.00 -> 63.1 mm, vias 0 -> 2
- net M1_0: track 0.00 -> 58.5 mm, vias 0 -> 2
- net FPGA_INIT_B: track 0.00 -> 51.4 mm, vias 0 -> 5
- net FPGA_CCLK: track 0.00 -> 48.3 mm, vias 0 -> 2
- net M2_0: track 0.00 -> 47.1 mm, vias 0 -> 2
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- added copper zone on B.Cu, net GND
- added copper zone on F.Cu, net GND
- added copper zone on In1.Cu, net GND
Other:
- board text added: "!!!"
- board text added: "+"
- board text added: "3V3"
- board text added: "GND"
- board text added: "M0"
- board text added: "M1"
- board text added: "M2"
- board text added: "PA1"
- board text added: "PC15"
- board text added: "Paulo Costa 11/09/2018"
